Commit message: Updated with customize URDF

File: src/my_robot_description/urdf/mobile_base.urdf.xacro (robot description, xacro)
@@ -3,12 +3,11 @@
      Commit Version: 1.6.0-4-g7f85cfe  Build Version: 1.6.7995.38578
      For more information, please see http://wiki.ros.org/sw_urdf_exporter -->
-<robot
-  name="Mobile_base">
-  <link
-    name="base_link">
-    <inertial>
-      <origin
-        xyz="-0.000106670270633216 0.0572278256509815 0.00180200077468832"
-        rpy="0 0 0" />
+<robot xmlns:xacro="http://www.ros.org/wiki/xacro">
+  <link name="base_footprint" />
+  <link name="base_link">
+    <inertial>
+      <origin
+        xyz="0 0 0"
+        rpy="-1.5708 0 -1.5708" />
       <mass
         value="0.600820640619417" />
@@ -24,8 +23,8 @@
       <origin
         xyz="0 0 0"
-        rpy="0 0 0" />
-      <geometry>
-        <mesh
-          filename="package://Mobile_base/meshes/base_link.STL" />
+        rpy="0 0 -1.5708" />
+      <geometry>
+        <mesh
+          filename="package://my_robot_description/meshes/base_link.STL" />
       </geometry>
       <material
@@ -38,17 +37,24 @@
       <origin
         xyz="0 0 0"
-        rpy="0 0 0" />
-      <geometry>
-        <mesh
-          filename="package://Mobile_base/meshes/base_link.STL" />
-      </geometry>
-    </collision>
-  </link>
-  <link
-    name="caster_wheel_link">
-    <inertial>
-      <origin
+        rpy="0 0 -1.5708" />
+      <geometry>
+        <mesh
+          filename="package://my_robot_description/meshes/base_link.STL" />
+      </geometry>
+    </collision>
+  </link>
+  <joint name="base_joint" type="fixed">
+      <parent link="base_footprint" />
+      <child link="base_link" />
+      <origin xyz="0 0 0.0445" rpy="0 0 0"/>
+  </joint>
+  <link name="caster_wheel_link">
+    <inertial>
+      <origin
+        xyz="0 0 0"
+        rpy="1.5708 0 1.5708" />
+      <!-- <origin
         xyz="6.9389E-18 0.0047803 4.1273E-18"
-        rpy="0 0 0" />
+        rpy="1.5708 0 1.5708" /> -->
       <mass
         value="0.0065128" />
@@ -64,8 +70,8 @@
       <origin
         xyz="0 0 0"
-        rpy="0 0 0" />
-      <geometry>
-        <mesh
-          filename="package://Mobile_base/meshes/caster_wheel_link.STL" />
+        rpy="1.5708 0 1.5708" />
+      <geometry>
+        <mesh
+          filename="package://my_robot_description/meshes/caster_wheel_link.STL" />
       </geometry>
       <material
@@ -78,17 +84,15 @@
       <origin
         xyz="0 0 0"
-        rpy="0 0 0" />
-      <geometry>
-        <mesh
-          filename="package://Mobile_base/meshes/caster_wheel_link.STL" />
-      </geometry>
-    </collision>
-  </link>
-  <joint
-    name="base_caster_wheel_joint"
-    type="fixed">
-    <origin
-      xyz="0 0.05 -0.04028"
-      rpy="1.5708 0 1.5708" />
+        rpy="1.5708 0 1.5708" />
+      <geometry>
+        <mesh
+          filename="package://my_robot_description/meshes/caster_wheel_link.STL" />
+      </geometry>
+    </collision>
+  </link>
+  <joint name="base_caster_wheel_joint" type="fixed">
+    <origin
+      xyz="0.05 0 -0.04028"
+      rpy="0 0 0" />
     <parent
       link="base_link" />
@@ -98,6 +102,5 @@
       xyz="0 0 0" />
   </joint>
-  <link
-    name="right_wheel_link">
+  <link name="right_wheel_link">
     <inertial>
       <origin
@@ -120,5 +123,5 @@
       <geometry>
         <mesh
-          filename="package://Mobile_base/meshes/right_wheel_link.STL" />
+          filename="package://my_robot_description/meshes/right_wheel_link.STL" />
       </geometry>
       <material
@@ -134,14 +137,12 @@
       <geometry>
         <mesh
-          filename="package://Mobile_base/meshes/right_wheel_link.STL" />
-      </geometry>
-    </collision>
-  </link>
-  <joint
-    name="base_right_wheel_joint"
-    type="continuous">
-    <origin
-      xyz="0.08975 -0.0445 -0.02"
-      rpy="1.5708 0 1.5708" />
+          filename="package://my_robot_description/meshes/right_wheel_link.STL" />
+      </geometry>
+    </collision>
+  </link>
+  <joint name="base_right_wheel_joint" type="continuous">
+    <origin
+      xyz="-0.0445 -0.08975 -0.02"
+      rpy="1.5708 0 0" />
     <parent
       link="base_link" />
@@ -149,8 +150,7 @@
       link="right_wheel_link" />
     <axis
-      xyz="0 0 1" />
-  </joint>
-  <link
-    name="left_wheel_link">
+      xyz="0 0 -1" />
+  </joint>
+  <link name="left_wheel_link">
     <inertial>
       <origin
@@ -173,5 +173,5 @@
       <geometry>
         <mesh
-          filename="package://Mobile_base/meshes/left_wheel_link.STL" />
+          filename="package://my_robot_description/meshes/left_wheel_link.STL" />
       </geometry>
       <material
@@ -187,5 +187,5 @@
       <geometry>
         <mesh
-          filename="package://Mobile_base/meshes/left_wheel_link.STL" />
+          filename="package://my_robot_description/meshes/left_wheel_link.STL" />
       </geometry>
     </collision>
@@ -195,6 +195,6 @@
     type="continuous">
     <origin
-      xyz="-0.08975 -0.0445 -0.02"
-      rpy="-1.5708 0 1.5708" />
+      xyz="-0.0445 0.08975 -0.02"
+      rpy="-1.5708 0 0" />
     <parent
       link="base_link" />
@@ -209,7 +209,7 @@
       <origin
         xyz="0 0 0"
-        rpy="0 0 0" />
-      <mass
-        value="0" />
+        rpy="1.5708 0 0" />
+      <mass
+        value="0.0" />
       <inertia
         ixx="0"
@@ -223,8 +223,8 @@
       <origin
         xyz="0 0 0"
-        rpy="0 0 0" />
-      <geometry>
-        <mesh
-          filename="package://Mobile_base/meshes/lidar_link.STL" />
+        rpy="1.5708 0 0" />
+      <geometry>
+        <mesh
+          filename="package://my_robot_description/meshes/lidar_link.STL" />
       </geometry>
       <material
@@ -237,17 +237,16 @@
       <origin
         xyz="0 0 0"
-        rpy="0 0 0" />
-      <geometry>
-        <mesh
-          filename="package://Mobile_base/meshes/lidar_link.STL" />
-      </geometry>
-    </collision>
-  </link>
-  <joint
-    name="base_lidar_joint"
-    type="fixed">
+        rpy="1.5708 0 0" />
+      <geometry>
+        <mesh
+          filename="package://my_robot_description/meshes/lidar_link.STL" />
+      </geometry>
+    </collision>
+  </link>
+  <joint name="base_lidar_joint" type="fixed">
     <origin
       xyz="3E-05 2.5E-05 0.20108"
-      rpy="1.5708 0 1.5708" />
+      rpy="0 0 0" />
+      <!-- rpy="1.5708 0 1.5708" /> -->
     <parent
       link="base_link" />

File: src/my_robot_description/urdf/my_robot.urdf.xacro (robot description, xacro)
@@ -5,5 +5,6 @@
     <xacro:arg name="baud" default="115200"/>
     <xacro:include filename="common_properties.xacro" />
-    <xacro:include filename="mobile_base.xacro" />
+    <!-- <xacro:include filename="mobile_base.xacro" /> -->
+    <xacro:include filename="mobile_base.urdf.xacro" />
     <xacro:include filename="mobile_base.ros2_control.xacro"/>
     <xacro:mobile_base_ros2_control
